Commit message: revised controller

File: ros2_ws2/src/my_agv2/urdf/AGV5.xacro.urdf (robot description, URDF)
Before this commit: robot AGV5, 36 links, 35 joints
Joints:
- joint TM_loader_joint: limit lower=-1.5 upper=0.3 effort=5 velocity=0.5 -> lower=0.0 upper=0.0 effort=5 velocity=0.5
- joint TM_slider_joint: limit lower=0 upper=0.41 effort=10 velocity=0.5 -> lower=0 upper=0 effort=10 velocity=0.5
- joint bot_slider_l_joint: limit lower=-0.07 upper=0.04 effort=1000000 velocity=10 -> lower=0.04 upper=0.04 effort=1000000 velocity=10
- joint bot_slider_r_joint: limit lower=-0.05 upper=0.088 effort=10000000 velocity=10 -> lower=-0.05 upper=-0.05 effort=10000000 velocity=10

Commit message: add lidar plugin and modify world

File: ros2_ws2/src/my_agv2/urdf/AGV5.xacro.urdf (robot description, URDF)
Before this commit: robot AGV5, 36 links, 35 joints
Links:
- added link lidar_link, mass 0.0001; collision sphere radius=0.01; visual sphere radius=0.02
Joints:
- added joint lidar_joint: type revolute, parent base_link, child lidar_link, origin xyz=0.0 0.6 0.0 rpy=1.57 0.0 0.0, axis 0 0 1, limit lower=0.0 upper=0.0 effort=100 velocity=0.1

Commit message: add imu sensor to model

File: ros2_ws2/src/my_agv2/urdf/AGV5.xacro.urdf (robot description, URDF)
Before this commit: robot AGV5, 37 links, 36 joints
Links:
- added link imu_link, mass 0.0001; collision sphere radius=0.01; visual sphere radius=0.02
Joints:
- added joint imu_joint: type revolute, parent base_link, child imu_link, origin xyz=0.0 0.0 0.0 rpy=0.0 0.0 0.0, axis 0 0 1, limit lower=0.0 upper=0.0 effort=100 velocity=0.1

Commit message: integrate with nav 2

File: ros2_ws2/src/my_agv2/urdf/AGV5.xacro.urdf (robot description, URDF)
Before this commit: robot AGV5, 38 links, 37 joints
Links:
- added link base_footprint, mass 0.0001
Joints:
- added joint base_footprint_joint: type fixed, parent base_footprint, child base_link, origin xyz=0 0 0 rpy=0 -1.57 0
- joint camera_1_joint: origin xyz=0.0 0.2 -0.44 rpy=0.0 2.17 1.57 -> xyz=0.0 0.2 -0.44 rpy=0.0 1.57 1.57
- joint camera_2_joint: origin xyz=0.0 0.2 0.44 rpy=3.14 -2.17 1.57 -> xyz=0.0 0.2 0.44 rpy=0.0 -1.57 -1.57
